File: main-board/quantizer-main.brd (EAGLE design)
At the start: 107.7 x 40 mm, 110 parts, among them IC1 PIC16F1829SOIC, IC2 TL074D, IC3 TL072D, IC4 4051D

Commit message: gdfgdf
Parts:
- removed C1: (no value), rcl:C0805
- added C22, C23: (no value), rcl:E2,5-7
- added C24: (no value), rcl:E2,5-5
- added C28, C9: (no value), rcl:C0805
- added D10, D9: MBR0520LT, diode:SOD123
- added F1, F2: (no value), microbuilder:PTC1210
- added IC8: REG1117, burr-brown:SOT223
- added L1, L2: (no value), wuerth-elektronik:0805
- added POWER: (no value), pinhead:2X05
- moved C8 231.0 mm to (91.4, 54.6), turned to 180 degrees
- moved IC4 213.0 mm to (82.5, 50.8), turned to 270 degrees
- moved J1 208.6 mm to (60.3, 67.9), flipped to the bottom, turned to 270 degrees
- moved C2 114.9 mm to (63.5, 50.2), turned to 180 degrees
- moved C3 100.6 mm to (44.5, 69.0)
- moved R9 91.7 mm to (50.0, 48.4), turned to 180 degrees
- moved C4 89.3 mm to (27.9, 70.2), turned to 180 degrees
- moved C5 85.0 mm to (105.4, 52.1)
- moved C7 35.6 mm to (52.8, 38.4)
- moved R10 30.2 mm to (50.0, 45.8), turned to 180 degrees
- moved C6 18.3 mm to (98.7, 49.0), turned to 0 degrees
- moved U$2 5.68 mm to (27.9, 63.5)
- moved R12 5.68 mm to (34.9, 64.8)
- moved R16 5.68 mm to (21.0, 64.8)
- moved R13 5.68 mm to (34.9, 62.2)
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Connections:
- new net N$41: D9.C, F1.P$2, L1.2
- new net N$42: D10.A, F2.P$2, L2.2
- new net N$63: F2.P$1, POWER.10, POWER.9
- new net N$75: F1.P$1, POWER.1, POWER.2
- net +12V: now also C22.+, C9.2, IC8.3, L1.1
- net +5V: now also C24.+, C28.2, IC8.2
- net -12V: now also C23.-, L2.1; no longer C1.1, IC2.11
- net CV_OUTA: now also U$1.7; no longer U$1.6
- net CV_OUTB: now also U$1.6; no longer U$1.7
- net CV_OUTC: now also U$1.9; no longer U$1.8
- net CV_OUTD: now also U$1.8; no longer U$1.9
- net GND: now also C22.-, C23.+, C24.-, C28.1, C9.1, D10.C, D9.A, IC2.11, IC8.1, POWER.3, POWER.4, POWER.5, POWER.6, POWER.7, POWER.8; no longer C1.2
Routing:
- net +5V: track 0.00 -> 192.1 mm, vias 0 -> 3
- net +12V: track 0.00 -> 120.0 mm, vias 0 -> 4
- net SWITCH: track 0.00 -> 101.7 mm, vias 0 -> 3
- net CVIN2: track 0.00 -> 84.3 mm, vias 0 -> 2
- net CVIN1: track 0.00 -> 81.8 mm, vias 0 -> 2
- net LED_B: track 0.00 -> 79.1 mm, vias 0 -> 1
- net LED_A: track 0.00 -> 78.7 mm, vias 0 -> 1
- net KBREAD3: track 0.00 -> 78.5 mm, vias 0 -> 1
- net N$10: track 0.00 -> 74.5 mm, vias 0 -> 1
- net MIDI_RX: track 0.00 -> 71.3 mm, vias 0 -> 2
- net CLKOUT: track 0.00 -> 70.3 mm, vias 0 -> 2
- net TRGOUT: track 0.00 -> 69.8 mm, vias 0 -> 2
- net N$9: track 0.00 -> 59.1 mm, vias 0 -> 1
- net DAC_SCL: track 0.00 -> 58.6 mm, vias 0 -> 3
- net N$5: track 0.00 -> 52.6 mm, vias 0 -> 1
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- added copper zone on layer 1, net GND
- added copper zone on layer 16, net GND

Commit message: dsfds
Parts:
- removed C22, C23: (no value), rcl:E2,5-7
- removed C24: (no value), rcl:E2,5-5
- removed C28: (no value), rcl:C0805
- removed U$1: MCP4728_QUAD_DAC, jason_eagle6:MSOP10
- removed U$2: NPIC6C596, jasons_stuff:SO16
- added C1, C10, C11, C12: (no value), rcl:C0805
- added IC5: REG1117, burr-brown:SOT223
- added IC6: 4051D, 40xx:SO16
- C7: device rcl:C0805 -> rcl:E2,5-5
- C8, C9: device rcl:C0805 -> rcl:E2,5-7
- IC1: value PIC16F1829SOIC -> NPIC6C596; device jason_eagle6:SO20W -> jasons_stuff:SO16
- IC2: value TL074D -> PIC16F1829SOIC; device linear:SO14 -> jason_eagle6:SO20W
- IC3: value TL072D -> TL074D; device linear:SO08 -> linear:SO14
- IC4: value 4051D -> MCP4728_QUAD_DAC; device 40xx:SO16 -> jason_eagle6:MSOP10
- IC8: value REG1117 -> TL072D; device burr-brown:SOT223 -> linear:SO08
- moved R31 93.8 mm to (111.6, 71.0)
- moved R33 93.2 mm to (111.8, 63.9)
- moved R27 89.0 mm to (103.0, 71.0), turned to 180 degrees
- moved R29 85.4 mm to (102.9, 63.9), turned to 180 degrees
- moved R32 83.2 mm to (111.8, 67.4)
- moved R28 82.8 mm to (102.9, 67.4), turned to 180 degrees
- moved R34 82.6 mm to (111.8, 60.3)
- moved R30 79.6 mm to (102.9, 60.3), turned to 180 degrees
- moved R21 54.3 mm to (56.4, 43.2)
- moved R19 49.0 mm to (56.4, 48.3), turned to 0 degrees
- moved R26 47.4 mm to (70.5, 40.6), turned to 180 degrees
- moved R23 47.0 mm to (70.5, 48.3), turned to 180 degrees
- moved R20 45.5 mm to (56.4, 45.7)
- moved R22 45.3 mm to (56.4, 40.6)
- moved R5 44.5 mm to (34.9, 67.3), turned to 0 degrees
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- renumbered OK1 to IC7, T1 to Q3, T2 to Q7, T3 to Q5, T4 to Q1, T5 to Q6, T6 to Q2, T7 to Q8, T8 to Q4, U$3 to D11, VR3 to VR1, VR4 to VR2
Connections:
- net +12V: now also C12.2, C4.1, C9.+, IC3.4, IC5.3, IC8.8, L2.1; no longer C2.1, C22.+, C9.2, IC2.4, IC3.8, IC8.3, L1.1
- net +5V: now also C1.1, C10.2, C2.1, C6.2, C7.+, D5.C, D7.C, IC1.7, IC2.1, IC4.1, IC5.2, IC6.16, R17.2, R18.2, R35.2; no longer C24.+, C28.2, C4.1, C7.1, C8.2, D2.C, D4.C, IC4.16, IC8.2, R10.2, R24.2, R9.2, U$1.1, U$2.1, U$2.7
- net -12V: now also C11.2, C8.-, IC8.4, L1.1; no longer C23.-, C6.2, IC3.4, L2.1
- net CLKIN: now also D4.C, D8.A, IC2.9, R12.2, R14.1; no longer D1.C, D2.A, IC1.9, R27.2, R28.1
- net CLKOUT: now also IC2.8, IC8.5; no longer IC1.8, IC3.5
- net CVIN1: now also D2.C, D6.A, IC6.13; no longer D7.C, D8.A, IC4.13
- net CVIN2: now also D1.C, D5.A, IC6.14; no longer D5.C, D6.A, IC4.14
- net CV_OUTA: now also IC3.3, IC4.7; no longer IC2.3, U$1.7
- net CV_OUTB: now also IC3.5, IC4.6; no longer IC2.5, U$1.6
- net CV_OUTC: now also IC3.10, IC4.9; no longer IC2.10, U$1.9
- net CV_OUTD: now also IC3.12, IC4.8; no longer IC2.12, U$1.8
- net DAC_SCL: now also IC2.16, IC4.2, R18.1; no longer IC1.16, R10.1, U$1.2
- net DAC_SDA: now also IC2.15, IC4.3, R17.1; no longer IC1.15, R9.1, U$1.3
- net GATEIN: now also D7.A, IC2.10, R11.2, R13.1; no longer D4.A, IC1.10, R29.2, R30.1
- net GND: now also C1.2, C10.1, C11.1, C12.1, C7.-, C8.+, C9.-, D10.A, D2.A, D4.A, D9.C, IC1.16, IC1.8, IC2.20, IC3.11, IC4.10, IC4.4, IC5.1, IC6.6, IC6.7, IC6.8, R13.2, R14.2, R15.2, R16.2, R20.2, R21.2, R24.1, R25.1, R36.2; no longer C22.-, C23.+, C24.-, C28.1, C7.2, C8.1, C9.1, D10.C, D5.A, D7.A, D9.A, IC1.20, IC2.11, IC4.6, IC4.7, IC4.8, IC8.1, R2.2, R22.2, R28.2, R30.2, R32.2, R34.2, R4.2, R7.1, R8.1, U$1.10, U$1.4, U$2.16, U$2.8
- net KBREAD1: now also IC6.15; no longer IC4.15
- net KBREAD2: now also IC6.12; no longer IC4.12
- net KBREAD3: now also IC2.6; no longer IC1.6
- net LED_A: now also IC2.19; no longer IC1.19
- net LED_B: now also IC2.18; no longer IC1.18
- net MIDI_RX: now also IC2.5, R35.1; no longer IC1.5, R24.1
- net MUXA: now also IC2.13, IC6.11; no longer IC1.13, IC4.11
- net MUXB: now also IC2.12, IC6.10; no longer IC1.12, IC4.10
- net MUXC: now also IC2.11, IC6.9; no longer IC1.11, IC4.9
- net MUXQ: now also IC2.14, IC6.3; no longer IC1.14, IC4.3
- net N$1: now also IC3.1, R19.2; no longer IC2.1, R1.2
- net N$10: now also IC3.14, R23.2; no longer IC2.14, R6.2
- net N$11: now also IC3.9, R25.2, R26.1; no longer IC2.9, R5.1, R7.2
- net N$12: now also IC3.13, R23.1, R24.2; no longer IC2.13, R6.1, R8.2
- net N$13: now also IC1.3, R1.2; no longer R15.2, U$2.3
- net N$14: now also IC1.4, R2.2; no longer R16.2, U$2.4
- net N$15: now also IC1.5, R3.2; no longer R17.2, U$2.5
- net N$16: now also IC1.6, R4.2; no longer R18.2, U$2.6
- net N$17: now also R5.2; no longer R11.2
- net N$18: now also R6.2; no longer R12.2
- net N$19: now also R7.2; no longer R13.2
- net N$2: now also IC3.2, R19.1, R20.1; no longer IC2.2, R1.1, R2.1
- net N$20: now also R8.2; no longer R14.2
- net N$21: now also IC1.14, R5.1; no longer R11.1, U$2.14
- net N$22: now also IC1.13, R6.1; no longer R12.1, U$2.13
- net N$23: now also IC1.12, R7.1; no longer R13.1, U$2.12
- net N$24: now also IC1.11, R8.1; no longer R14.1, U$2.11
- net N$26: now also R29.1; no longer R19.1
- net N$27: now also R37.1; no longer R20.1
- net N$28: now also R33.2; no longer R26.2
- net N$3: now also R1.1; no longer R15.1
- net N$30: now also R27.1; no longer R21.1
- net N$31: now also R37.2; no longer R20.2
- net N$32: now also R33.1; no longer R26.1
- net N$33: now also R31.2; no longer R23.2
- net N$34: now also R31.1; no longer R23.1
- net N$37: now also R28.1; no longer R25.1
- net N$38: now also R32.2; no longer R35.2
- net N$39: now also R32.1; no longer R35.1
- net N$4: now also IC3.6, R21.1, R22.1; no longer IC2.6, R3.1, R4.1
- net N$41: now also D10.C, F2.P$2, L2.2; no longer D9.C, F1.P$2, L1.2
- net N$42: now also D9.A, F1.P$2, L1.2; no longer D10.A, F2.P$2, L2.2
- net N$44: now also R30.1; no longer R36.1
- net N$45: now also R34.2; no longer R37.2
- net N$46: now also R12.1; no longer R27.1
- net N$47: now also R36.1; no longer R22.1
- net N$48: now also R34.1; no longer R37.1
- net N$5: now also IC3.7, R22.2; no longer IC2.7, R3.2
- net N$50: now also R11.1; no longer R29.1
- net N$53: now also R9.1; no longer R31.1
- net N$54: now also R9.2; no longer R31.2
- net N$55: now also R15.1; no longer R32.1
- net N$56: now also R10.1; no longer R33.1
- net N$57: now also R10.2; no longer R33.2
- net N$58: now also R16.1; no longer R34.1
- net N$6: now also R2.1; no longer R16.1
- net N$60: now also IC8.1, IC8.2, R39.1; no longer IC3.1, IC3.2, R38.1
- net N$61: now also IC8.6, IC8.7, R38.1; no longer IC3.6, IC3.7, R39.1
- net N$63: now also F1.P$1; no longer F2.P$1
- net N$64: now also R39.2; no longer R38.2
- net N$65: now also R38.2; no longer R39.2
- net N$7: now also R3.1; no longer R17.1
- net N$75: now also F2.P$1; no longer F1.P$1
- net N$8: now also R4.1; no longer R18.1
- net N$9: now also IC3.8, R26.2; no longer IC2.8, R5.2
- net SRC1: now also IC6.1, R29.2; no longer IC4.1, R19.2
- net SRC2: now also IC6.5, R27.2; no longer IC4.5, R21.2
- net SRC3: now also IC6.2, R28.2; no longer IC4.2, R25.2
- net SRC4: now also IC6.4, R30.2; no longer IC4.4, R36.2
- net SR_DATA: now also IC1.2, IC2.17; no longer IC1.17, U$2.2
- net SR_SHIFT: now also IC1.15, IC2.2; no longer IC1.2, U$2.15
- net SR_STORE: now also IC1.10, IC2.3; no longer IC1.3, U$2.10
- net SWITCH: now also IC2.4; no longer IC1.4
- net TRGOUT: now also IC2.7, IC8.3; no longer IC1.7, IC3.3
Other:
- board text added: "+12V"
- board text added: "-12V"
