File: main-board/quantizer-main.sch (EAGLE design)
At the start: 110 parts, among them IC1 PIC16F1829SOIC, IC2 TL074D, IC3 TL072D, IC4 4051D

Commit message: gdfgdf
Parts:
- removed C1: (no value), rcl:C-EUC0805
- added C22, C23: (no value), rcl:CPOL-EUE2.5-7
- added C24: (no value), rcl:CPOL-EUE2.5-5
- added C28, C9: (no value), rcl:C-EUC0805
- added D10, D9: MBR0520LT, diode:MBR0520LT
- added F1, F2: (no value), microbuilder:PTC1210
- added IC8: REG1117, burr-brown:REG1117
- added L1, L2: (no value), wuerth-elektronik:WE-CBF_0805
- added POWER: (no value), pinhead:PINHD-2X5
Connections:
- new net N$41: D9.C, F1.2, L1.2
- new net N$42: D10.A, F2.2, L2.2
- new net N$63: F2.1, POWER.10, POWER.9
- new net N$75: F1.1, POWER.1, POWER.2
- net +12V: now also C22.+, C9.2, IC8.VIN, L1.1
- net +5V: now also C24.+, C28.2, IC8.VOUT
- net -12V: now also C23.-, L2.1; no longer C1.1, IC2P.V-
- net CV_OUTA: now also U$1.VOUTB; no longer U$1.VOUTA
- net CV_OUTB: now also U$1.VOUTA; no longer U$1.VOUTB
- net CV_OUTC: now also U$1.VOUTD; no longer U$1.VOUTC
- net CV_OUTD: now also U$1.VOUTC; no longer U$1.VOUTD
- net GND: now also C22.-, C23.+, C24.-, C28.1, C9.1, D10.C, D9.A, IC2P.V-, IC8.GND, POWER.3, POWER.4, POWER.5, POWER.6, POWER.7, POWER.8; no longer C1.2
Other:
- note added: "CLOCK/GATE OUTPUT BUFFERS"
- note added: "CLOCK/TRIG INPUTS"
- note added: "CV DAC"
- note added: "CV OUTPUT BUFFERS"
- note added: "I/O MULTIPLEXER"
- note added: "LED SOURCE DRIVERS"
- note added: "MIDI INPUT"
- note added: "PITCH CV INPUTS"
- note added: "POWER SUPPLY"
- note added: "PROCESSOR"
- note added: "SINK SHIFT REGISTER"
- moved on the sheet: C2, C3, C4, C5, C6, C7, C8, CLKOUT, CLK_IN, CVIN1, CVIN2, CVOUT1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

Commit message: dsfds
Parts:
- removed C22, C23: (no value), rcl:CPOL-EUE2.5-7
- removed C24: (no value), rcl:CPOL-EUE2.5-5
- removed C28: (no value), rcl:C-EUC0805
- removed U$1: MCP4728_QUAD_DAC, jason_eagle6:MCP4728_QUAD_DAC
- removed U$2: NPIC6C596, jasons_stuff:NPIC6C596
- added C1, C10, C11, C12: (no value), rcl:C-EUC0805
- added IC5: REG1117, burr-brown:REG1117
- added IC6: 4051D, 40xx:4051D
- C7: device rcl:C-EUC0805 -> rcl:CPOL-EUE2.5-5
- C8, C9: device rcl:C-EUC0805 -> rcl:CPOL-EUE2.5-7
- IC1: value PIC16F1829SOIC -> NPIC6C596; device jason_eagle6:PIC16F1829SOIC -> jasons_stuff:NPIC6C596
- IC2: value TL074D -> PIC16F1829SOIC; device linear:TL074D -> jason_eagle6:PIC16F1829SOIC
- IC3: value TL072D -> TL074D; device linear:TL072D -> linear:TL074D
- IC4: value 4051D -> MCP4728_QUAD_DAC; device 40xx:4051D -> jason_eagle6:MCP4728_QUAD_DAC
- IC8: value REG1117 -> TL072D; device burr-brown:REG1117 -> linear:TL072D
- renumbered OK1 to IC7, T1 to Q3, T2 to Q7, T3 to Q5, T4 to Q1, T5 to Q6, T6 to Q2, T7 to Q8, T8 to Q4, U$3 to D11, VR3 to VR1, VR4 to VR2
Connections:
- net +12V: now also C12.2, C4.1, C9.+, IC5.VIN, IC8P.V+, L2.1; no longer C2.1, C22.+, C9.2, IC2P.V+, IC8.VIN, L1.1
- net +5V: now also C1.1, C10.2, C2.1, C6.2, C7.+, D5.C, D7.C, IC1.MR#, IC1.VCC, IC2.VDD, IC4.VDD, IC5.VOUT, IC6P.VCC, R17.2, R18.2, R35.2; no longer C24.+, C28.2, C4.1, C7.1, C8.2, D2.C, D4.C, IC1.VDD, IC4P.VCC, IC8.VOUT, R10.2, R24.2, R9.2, U$1.VDD, U$2.MR#, U$2.VCC
- net -12V: now also C11.2, C8.-, IC8P.V-, L1.1; no longer C23.-, C6.2, IC3P.V-, L2.1
- net CLKIN: now also D4.C, D8.A, IC2.RC7, R12.2, R14.1; no longer D1.C, D2.A, IC1.RC7, R27.2, R28.1
- net CLKOUT: now also IC2.RC6, IC8B.+IN; no longer IC1.RC6, IC3B.+IN
- net CVIN1: now also D2.C, D6.A, IC6A.X0; no longer D7.C, D8.A, IC4A.X0
- net CVIN2: now also D1.C, D5.A, IC6A.X1; no longer D5.C, D6.A, IC4A.X1
- net CV_OUTA: now also IC3A.+IN, IC4.VOUTB; no longer IC2A.+IN, U$1.VOUTB
- net CV_OUTB: now also IC3B.+IN, IC4.VOUTA; no longer IC2B.+IN, U$1.VOUTA
- net CV_OUTC: now also IC3C.+IN, IC4.VOUTD; no longer IC2C.+IN, U$1.VOUTD
- net CV_OUTD: now also IC3D.+IN, IC4.VOUTC; no longer IC2D.+IN, U$1.VOUTC
- net DAC_SCL: now also IC2.RC0, IC4.SCL, R18.1; no longer IC1.RC0, R10.1, U$1.SCL
- net DAC_SDA: now also IC2.RC1, IC4.SDA, R17.1; no longer IC1.RC1, R9.1, U$1.SDA
- net GATEIN: now also D7.A, IC2.RB7, R11.2, R13.1; no longer D4.A, IC1.RB7, R29.2, R30.1
- net GND: now also C1.2, C10.1, C11.1, C12.1, C7.-, C8.+, C9.-, D10.A, D2.A, D4.A, D9.C, IC1.GND, IC1.OE#, IC2.VSS, IC3P.V-, IC4.LDAC#, IC4.VSS, IC5.GND, IC6A.INH, IC6P.GND, IC6P.VEE, R13.2, R14.2, R15.2, R16.2, R20.2, R21.2, R24.1, R25.1, R36.2; no longer C22.-, C23.+, C24.-, C28.1, C7.2, C8.1, C9.1, D10.C, D5.A, D7.A, D9.A, IC1.VSS, IC2P.V-, IC4A.INH, IC4P.GND, IC4P.VEE, IC8.GND, R2.2, R22.2, R28.2, R30.2, R32.2, R34.2, R4.2, R7.1, R8.1, U$1.LDAC#, U$1.VSS, U$2.GND, U$2.OE#
- net KBREAD1: now also IC6A.X2; no longer IC4A.X2
- net KBREAD2: now also IC6A.X3; no longer IC4A.X3
- net KBREAD3: now also IC2.RC4; no longer IC1.RC4
- net LED_A: now also IC2.RA0; no longer IC1.RA0
- net LED_B: now also IC2.RA1; no longer IC1.RA1
- net MIDI_RX: now also IC2.RC5, R35.1; no longer IC1.RC5, R24.1
- net MUXA: now also IC2.RB4, IC6A.A; no longer IC1.RB4, IC4A.A
- net MUXB: now also IC2.RB5, IC6A.B; no longer IC1.RB5, IC4A.B
- net MUXC: now also IC2.RB6, IC6A.C; no longer IC1.RB6, IC4A.C
- net MUXQ: now also IC2.RC2, IC6A.X; no longer IC1.RC2, IC4A.X
- net N$1: now also IC3A.OUT, R19.2; no longer IC2A.OUT, R1.2
- net N$10: now also IC3D.OUT, R23.2; no longer IC2D.OUT, R6.2
- net N$11: now also IC3C.-IN, R25.2, R26.1; no longer IC2C.-IN, R5.1, R7.2
- net N$12: now also IC3D.-IN, R23.1, R24.2; no longer IC2D.-IN, R6.1, R8.2
- net N$13: now also IC1.Q0, R1.2; no longer R15.2, U$2.Q0
- net N$14: now also IC1.Q1, R2.2; no longer R16.2, U$2.Q1
- net N$15: now also IC1.Q2, R3.2; no longer R17.2, U$2.Q2
- net N$16: now also IC1.Q3, R4.2; no longer R18.2, U$2.Q3
- net N$17: now also R5.2; no longer R11.2
- net N$18: now also R6.2; no longer R12.2
- net N$19: now also R7.2; no longer R13.2
- net N$2: now also IC3A.-IN, R19.1, R20.1; no longer IC2A.-IN, R1.1, R2.1
- net N$20: now also R8.2; no longer R14.2
- net N$21: now also IC1.Q7, R5.1; no longer R11.1, U$2.Q7
- net N$22: now also IC1.Q6, R6.1; no longer R12.1, U$2.Q6
- net N$23: now also IC1.Q5, R7.1; no longer R13.1, U$2.Q5
- net N$24: now also IC1.Q4, R8.1; no longer R14.1, U$2.Q4
- net N$26: now also R29.1; no longer R19.1
- net N$27: now also R37.1; no longer R20.1
- net N$28: now also R33.2; no longer R26.2
- net N$3: now also R1.1; no longer R15.1
- net N$30: now also R27.1; no longer R21.1
- net N$31: now also R37.2; no longer R20.2
- net N$32: now also R33.1; no longer R26.1
- net N$33: now also R31.2; no longer R23.2
- net N$34: now also R31.1; no longer R23.1
- net N$37: now also R28.1; no longer R25.1
- net N$38: now also R32.2; no longer R35.2
- net N$39: now also R32.1; no longer R35.1
- net N$4: now also IC3B.-IN, R21.1, R22.1; no longer IC2B.-IN, R3.1, R4.1
- net N$41: now also D10.C, F2.2, L2.2; no longer D9.C, F1.2, L1.2
- net N$42: now also D9.A, F1.2, L1.2; no longer D10.A, F2.2, L2.2
- net N$44: now also R30.1; no longer R36.1
- net N$45: now also R34.2; no longer R37.2
- net N$46: now also R12.1; no longer R27.1
- net N$47: now also R36.1; no longer R22.1
- net N$48: now also R34.1; no longer R37.1
- net N$5: now also IC3B.OUT, R22.2; no longer IC2B.OUT, R3.2
- net N$50: now also R11.1; no longer R29.1
- net N$53: now also R9.1; no longer R31.1
- net N$54: now also R9.2; no longer R31.2
- net N$55: now also R15.1; no longer R32.1
- net N$56: now also R10.1; no longer R33.1
- net N$57: now also R10.2; no longer R33.2
- net N$58: now also R16.1; no longer R34.1
- net N$6: now also R2.1; no longer R16.1
- net N$60: now also IC8A.-IN, IC8A.OUT, R39.1; no longer IC3A.-IN, IC3A.OUT, R38.1
- net N$61: now also IC8B.-IN, IC8B.OUT, R38.1; no longer IC3B.-IN, IC3B.OUT, R39.1
- net N$63: now also F1.1; no longer F2.1
- net N$64: now also R39.2; no longer R38.2
- net N$65: now also R38.2; no longer R39.2
- net N$7: now also R3.1; no longer R17.1
- net N$75: now also F2.1; no longer F1.1
- net N$8: now also R4.1; no longer R18.1
- net N$9: now also IC3C.OUT, R26.2; no longer IC2C.OUT, R5.2
- net SRC1: now also IC6A.X4, R29.2; no longer IC4A.X4, R19.2
- net SRC2: now also IC6A.X5, R27.2; no longer IC4A.X5, R21.2
- net SRC3: now also IC6A.X6, R28.2; no longer IC4A.X6, R25.2
- net SRC4: now also IC6A.X7, R30.2; no longer IC4A.X7, R36.2
- net SR_DATA: now also IC1.DS, IC2.RA2; no longer IC1.RA2, U$2.DS
- net SR_SHIFT: now also IC1.SHCP, IC2.RA5; no longer IC1.RA5, U$2.SHCP
- net SR_STORE: now also IC1.STCP, IC2.RA4; no longer IC1.RA4, U$2.STCP
- net SWITCH: now also IC2.RA3/MC#; no longer IC1.RA3/MC#
- net TRGOUT: now also IC2.RC3, IC8A.+IN; no longer IC1.RC3, IC3A.+IN
Other:
- moved on the sheet: C2, C3, C4, C5, C6, D1, D10, D2, D4, D5, D6, D7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
